File: stepstick-breakout.kicad_pcb (KiCad board)
At the start: 2 copper layers, 15.2 x 20.3 mm, 4 parts, among them J1 Conn_01x08, J2 Conn_01x08, J3 Conn_01x06, J4 Conn_01x02

Commit message: Rev 1.0
First Batch
Parts:
- added G***: LOGO, LOGO, B.Cu at (111.8, 76.2)
Routing:
- net /En: track 0.00 -> 13.6 mm
- net /Vm: track 0.00 -> 12.5 mm
- net /DIAG: track 0.00 -> 10.1 mm
- net /Dir: track 0.00 -> 5.61 mm
- net /Step: track 0.00 -> 5.59 mm
- added copper zone on B.Cu, net /GND
Other:
- outline, holes or cut-outs redrawn
- board text added: "Electric Magpie"
- board text added: "Stepstick-Breakout v1.0 May 2024"

Commit message: v1.1
Widened JST-XH mounting holes to theoretically support a 2.54mm pitch screw terminal array
Other:
- board text added: "Stepstick-Breakout v1.1 May 2024"
- board text removed: "Stepstick-Breakout v1.0 May 2024"
Changed lines of the file:
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@@
 		(pad "1" thru_hole roundrect
 			(at 0 0 270)
-			(size 1.7 1.95)
-			(drill 0.95)
+			(size 1.8 2.05)
+			(drill 1.05)
 			(layers "*.Cu" "*.Mask")
 			(remove_unused_layers no)
@@
 		(pad "2" thru_hole oval
 			(at 2.5 0 270)
-			(size 1.7 1.95)
-			(drill 0.95)
+			(size 1.75 2)
+			(drill 1)
 			(layers "*.Cu" "*.Mask")
 			(remove_unused_layers no)
@@
 		(pad "5" thru_hole oval
 			(at 10 0 270)
-			(size 1.7 1.95)
-			(drill 0.95)
+			(size 1.75 2)
+			(drill 1)
 			(layers "*.Cu" "*.Mask")
 			(remove_unused_layers no)
@@
 		(pad "6" thru_hole oval
 			(at 12.5 0 270)
-			(size 1.7 1.95)
-			(drill 0.95)
+			(size 1.8 2.05)
+			(drill 1.05)
 			(layers "*.Cu" "*.Mask")
 			(remove_unused_layers no)
@@
 		)
 	)
-	(gr_text "Stepstick-Breakout\nv1.0 May 2024"
+	(gr_text "Stepstick-Breakout\nv1.1 May 2024"
 		(at 111.506 66.04 90)
 		(layer "B.SilkS")
@@
 			(justify mirror)
 		)
-		(render_cache "Stepstick-Breakout\nv1.0 May 2024" 90
+		(render_cache "Stepstick-Breakout\nv1.1 May 2024" 90
 			(polygon
 				(pts
@@
 			(polygon
 				(pts
-					(xy 112.289425 63.332764) (xy 112.342198 63.334102) (xy 112.407628 63.338382) (xy 112.467421 63.345517)
-					(xy 112.521576 63.355505) (xy 112.581342 63.372003) (xy 112.632299 63.39296) (xy 112.681819 63.423994)
-					(xy 112.695762 63.435666) (xy 112.732194 63.473392) (xy 112.76053 63.515183) (xy 112.780769 63.56104)
-					(xy 112.792913 63.610962) (xy 112.796961 63.664949) (xy 112.794398 63.709729) (xy 112.784558 63.759258)
-					(xy 112.763749 63.811242) (xy 112.732894 63.856981) (xy 112.691993 63.896473) (xy 112.648136 63.925426)
-					(xy 112.596281 63.949472) (xy 112.549039 63.965175) (xy 112.496679 63.977738) (xy 112.439201 63.98716)
-					(xy 112.376605 63.993441) (xy 112.3263 63.996091) (xy 112.273115 63.996975) (xy 112.237284 63.996585)
-					(xy 112.185967 63.994539) (xy 112.122075 63.989084) (xy 112.063365 63.980511) (xy 112.009834 63.968821)
-					(xy 111.950205 63.949824) (xy 111.89867 63.925956) (xy 111.855229 63.897218) (xy 111.81905 63.863497)
-					(xy 111.786303 63.818421) (xy 111.763743 63.767171) (xy 111.752515 63.718328) (xy 111.748772 63.664949)
-					(xy 111.923471 63.664949) (xy 111.924851 63.682195) (xy 111.945556 63.727979) (xy 111.984142 63.756184)
-					(xy 112.033153 63.773887) (xy 112.061474 63.780043) (xy 112.111205 63.78627) (xy 112.165941 63.789861)
-					(xy 112.221194 63.79156) (xy 112.273115 63.792002) (xy 112.315262 63.791684) (xy 112.372521 63.790015)
-					(xy 112.422626 63.786915) (xy 112.47204 63.78149) (xy 112.521266 63.771654) (xy 112.559 63.758486)
-					(xy 112.600178 63.728475) (xy 112.60984 63.71399) (xy 112.622263 63.664949) (xy 112.620914 63.647687)
-					(xy 112.600674 63.60167) (xy 112.562367 63.573666) (xy 112.513573 63.556011) (xy 112.485159 63.549854)
-					(xy 112.435304 63.543627) (xy 112.380459 63.540036) (xy 112.325114 63.538338) (xy 112.273115 63.537896)
-					(xy 112.231015 63.538214) (xy 112.173767 63.539883) (xy 112.123604 63.542983) (xy 112.074034 63.548408)
-					(xy 112.024468 63.558244) (xy 111.986733 63.571412) (xy 111.945556 63.601422) (xy 111.935894 63.615908)
-					(xy 111.923471 63.664949) (xy 111.748772 63.664949) (xy 111.751335 63.620098) (xy 111.761176 63.570498)
-					(xy 111.781985 63.518455) (xy 111.81284 63.47268) (xy 111.85374 63.433176) (xy 111.897562 63.404223)
-					(xy 111.949307 63.380177) (xy 111.996409 63.364474) (xy 112.048583 63.351912) (xy 112.105828 63.34249)
-					(xy 112.168145 63.336208) (xy 112.218211 63.333558) (xy 112.27113 63.332675)
+					(xy 112.78108 63.83518) (xy 112.78108 63.639141) (xy 112.034146 63.639141) (xy 112.072561 63.597495)
+					(xy 112.107032 63.553145) (xy 112.137561 63.506091) (xy 112.164146 63.456332) (xy 112.186788 63.403868)
+					(xy 112.193459 63.385779) (xy 112.002879 63.385779) (xy 111.983211 63.435012) (xy 111.958134 63.481559)
+					(xy 111.929976 63.524714) (xy 111.909574 63.552537) (xy 111.873654 63.59404) (xy 111.834881 63.628471)
+					(xy 111.793253 63.655829) (xy 111.748772 63.676116) (xy 111.748772 63.83518)
 				)
 			)
@@
 	)
 	(zone
-		(net 14)
-		(net_name "/Step")
+		(net 2)
+		(net_name "/Vm")
 		(layer "F.Cu")
 		(name "$teardrop_padvia$")
 		(hatch full 0.1)
-		(priority 30001)
+		(priority 30003)
 		(attr
 			(teardrop
@@
 		(polygon
 			(pts
-				(xy 106.141333 63.206) (xy 106.141333 63.714) (xy 107.659173 64.293667) (xy 107.951 63.46) (xy 107.659173 62.626333)
+				(xy 113.87 77.089) (xy 113.87 77.851) (xy 115.244719 78.255298) (xy 115.571 77.47) (xy 115.244719 76.684702)
 			)
 		)
 	)
 	(zone
-		(net 16)
-		(net_name "/DIAG")
+		(net 14)
+		(net_name "/Step")
 		(layer "F.Cu")
 		(name "$teardrop_padvia$")
 		(hatch full 0.1)
-		(priority 30009)
+		(priority 30001)
 		(attr
 			(teardrop
@@
 		(polygon
 			(pts
-				(xy 106.299 76.033025) (xy 105.791 76.033025) (xy 104.808959 76.868959) (xy 105.41 77.471) (xy 106.26 77.47)
+				(xy 106.091813 63.206) (xy 106.091813 63.714) (xy 107.654296 64.318187) (xy 107.951 63.46) (xy 107.654296 62.601813)
 			)
 		)
 	)
 	(zone
-		(net 8)
-		(net_name "/En")
+		(net 16)
+		(net_name "/DIAG")
 		(layer "F.Cu")
 		(name "$teardrop_padvia$")
 		(hatch full 0.1)
-		(priority 30003)
+		(priority 30009)
 		(attr
 			(teardrop
@@
 		(polygon
 			(pts
-				(xy 106.517363 67.033427) (xy 106.876573 67.392637) (xy 108.373276 66.738804) (xy 107.950707 65.959293)
-				(xy 106.991333 65.794173)
+				(xy 106.299 76.033025) (xy 105.791 76.033025) (xy 104.808959 76.868959) (xy 105.41 77.471) (xy 106.26 77.47)
 			)
 		)
@@
 		(polygon
 			(pts
-				(xy 109.758667 71.341) (xy 109.758667 70.579) (xy 108.240827 70.126333) (xy 107.949 70.96) (xy 108.240827 71.793667)
+				(xy 109.808187 71.341) (xy 109.808187 70.579) (xy 108.245704 70.101813) (xy 107.949 70.96) (xy 108.245704 71.818187)
 			)
 		)
@@
 		(name "$teardrop_padvia$")
 		(hatch full 0.1)
-		(priority 30004)
+		(priority 30005)
 		(attr
 			(teardrop
@@
 	)
 	(zone
-		(net 2)
-		(net_name "/Vm")
+		(net 13)
+		(net_name "/Dir")
 		(layer "F.Cu")
 		(name "$teardrop_padvia$")
@@
 		(polygon
 			(pts
-				(xy 113.87 77.089) (xy 113.87 77.851) (xy 115.244719 78.255298) (xy 115.571 77.47) (xy 115.244719 76.684702)
+				(xy 106.025 60.706) (xy 106.025 61.214) (xy 107.088407 61.83985) (xy 107.951 60.96) (xy 107.088407 60.08015)
 			)
 		)
 	)
 	(zone
-		(net 8)
-		(net_name "/En")
+		(net 13)
+		(net_name "/Dir")
 		(layer "F.Cu")
 		(name "$teardrop_padvia$")
 		(hatch full 0.1)
-		(priority 30007)
+		(priority 30006)
 		(attr
 			(teardrop
@@
 		(polygon
 			(pts
-				(xy 104.251686 76.447524) (xy 103.892476 76.088314) (xy 102.544719 76.684702) (xy 102.869293 77.470707)
-				(xy 103.655298 77.795281)
+				(xy 104.141435 60.685645) (xy 104.500645 60.326435) (xy 103.72 59.192611) (xy 102.869293 59.689293)
+				(xy 102.647858 60.54)
 			)
 		)
 	)
 	(zone
-		(net 13)
-		(net_name "/Dir")
+		(net 8)
+		(net_name "/En")
 		(layer "F.Cu")
 		(name "$teardrop_padvia$")
 		(hatch full 0.1)
-		(priority 30005)
+		(priority 30004)
 		(attr
 			(teardrop
@@
 		(polygon
 			(pts
-				(xy 106.125 60.706) (xy 106.125 61.214) (xy 107.129329 61.79097) (xy 107.951 60.96) (xy 107.129329 60.12903)
+				(xy 106.517363 67.033427) (xy 106.876573 67.392637) (xy 108.373276 66.738804) (xy 107.950707 65.959293)
+				(xy 106.991333 65.794173)
 			)
 		)
 	)
 	(zone
-		(net 13)
-		(net_name "/Dir")
+		(net 8)
+		(net_name "/En")
 		(layer "F.Cu")
 		(name "$teardrop_padvia$")
 		(hatch full 0.1)
-		(priority 30006)
+		(priority 30007)
 		(attr
 			(teardrop
@@
 		(polygon
 			(pts
-				(xy 104.141435 60.685645) (xy 104.500645 60.326435) (xy 103.72 59.192611) (xy 102.869293 59.689293)
-				(xy 102.647858 60.54)
+				(xy 104.251686 76.447524) (xy 103.892476 76.088314) (xy 102.544719 76.684702) (xy 102.869293 77.470707)
+				(xy 103.655298 77.795281)
 			)
 		)
